File: PCB_Eagle/vA-ESP32.brd (EAGLE design)
At the start: 15 x 35 mm, 68 parts, among them U1 25Q32, U14 ESP32, U18 M24SR04, U2 LTC4054, U8 LIS3DH, U9 MCP170x-3.0, X3 I2C-SMD-SWATCH-I2C-5, Y1 32.768, Y2 26MHz

Commit message: v
Parts:
- removed CP5, CP6: (no value), !ht3_connectors:CP-1-C08MM
- removed D1: BAT54C-SOT323, !ht3_diode:SOT323
- removed D2: BAT54A-SOT323, !ht3_diode:SOT323
- removed LCD1: (no value), !ht3_modules:UG-2832HSWEG02_WRAPUNDER
- removed R19: 10K, !ht3_passive:R0603
- removed R20, R21: 4.7K, !ht3_passive:R0603
- removed R5: 0, !ht3_passive:R0402
- removed R6: 100, !ht3_passive:R0402
- removed U18: M24SR04, !ht3_ic:TSSOP08
- added C11, C5: 270pF, !ht3_passive:C0603
- added C12: 100nF, !ht3_passive:C0603
- added C16, C18: 270pF, !ht3_passive:C0805
- added LOGO1: LOGO6, !ht3_misc:LOGO_OMEGA
- added Q4: IRLML6401TR, !ht3_transistor:SOT23-3-1
- added VD1: (no value), !ht3_diode:SOD523
- C1: device !ht3_passive:C0402 -> !ht3_passive:C0603
- C40: value 10nF -> 100nF; device !ht3_passive:C0603 -> !ht3_passive:C0402
- D3: value 5.1V -> SS34; device !ht3_diode:SOD80C -> !ht3_diode:SOD123
- R4: value 0 -> 560K; device !ht3_passive:R0402 -> !ht3_passive:R0603
- moved FIDUCIAL1 31.5 mm to (14.0, 32.0), turned to 180 degrees
- moved C6 24.0 mm to (3.30, 1.20), turned to 90 degrees
- moved OLED1 23.2 mm to (7.50, 25.8), flipped to the bottom
- moved RA4 22.1 mm to (2.30, 17.0), turned to 90 degrees
- moved Y1 21.6 mm to (1.50, 2.30), turned to 270 degrees
- moved R2 20.8 mm to (13.8, 22.1)
- moved RA3 18.7 mm to (7.50, 1.30), turned to 0 degrees
- moved D3 18.6 mm to (3.00, 30.0), turned to 0 degrees
- moved C8 17.8 mm to (3.30, 3.00), turned to 270 degrees
- moved C14 16.4 mm to (7.00, 17.2), turned to 0 degrees
- moved CP7 15.8 mm to (10.8, 16.5), turned to 90 degrees
- moved CP4 15.7 mm to (1.00, 12.5), turned to 180 degrees
- moved R12 15.2 mm to (1.10, 22.9), turned to 180 degrees
- moved C25 14.6 mm to (3.50, 15.1), turned to 0 degrees
- moved C49 14.3 mm to (0.90, 10.9), turned to 270 degrees
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Connections:
- removed net IO26: U14.15
- removed net N$21: CP5.1, D1.1, D2.2
- removed net N$24: CP6.1, D1.2, D2.1
- removed net N$28: RA3.7, RA3.8
- removed net N$33: U18.1
- removed net N$70: U18.3
- removed net N$71: U18.2
- removed net N$8: U18.7
- removed net SCREEN_LED: Q2.1, R21.2, RA3.3, U14.22
- removed net VBREF: LCD1.6
- removed net VCC: LCD1.14
- removed net VCOMH: LCD1.13
- removed net VSS: LCD1.7
- new net IO2: Q2.1, RA3.3, U14.22
- new net N$10: C5.2, OLED1.1
- new net N$11: C12.1, C18.1, OLED1.14
- new net N$12: C16.1, OLED1.13
- new net N$14: OLED1.12, R4.2
- new net VBAT1: Q4.3
- net +5V: now also D3.A, Q4.1; no longer D3.C, R6.2
- net EN: now also RA3.1; no longer R19.2
- net GND: now also C12.2, C16.2, C18.2, OLED1.7, R4.1; no longer D2.3, D3.A, R21.1, U18.4
- net I2C_SCL: now also OLED1.10; no longer U18.6
- net I2C_SDA: now also OLED1.11; no longer U18.5
- net IO0: now also RA4.4; no longer R20.1
- net MOTOR: now also U14.15
- net N$1: now also C11.2, OLED1.3; no longer R4.2, U14.12
- net N$22: now also VD1.A
- net N$23: now also VD1.C
- net N$3: now also C11.1, OLED1.4; no longer D1.3, R6.1
- net N$5: now also C5.1, OLED1.2; no longer R5.2, U14.13
- net OSC32_I: now also U14.12; no longer R4.1
- net OSC32_O: now also U14.13; no longer R5.1
- net SCREEN_RES: now also OLED1.9
- net VBAT: now also D3.C, Q4.2; no longer LCD1.5
- net VBAT_ADC: no longer U14.10
- net VDD: now also OLED1.5, OLED1.8, RA3.7, RA3.8, RA4.5; no longer LCD1.8, R19.1, R20.2, U18.8
Routing:
- net GND: track 1.36 -> 34.7 mm, vias 20 -> 24
- net IO4: track 31.8 -> 4.30 mm
- net N$23: track 0.00 -> 25.5 mm
- net /IRQ: track 2.04 -> 26.9 mm, vias 0 -> 2
- net VDD: track 46.5 -> 70.6 mm, vias 6 -> 8
- net SCREEN_RES: track 6.10 -> 26.5 mm
- net VBAT: track 14.3 -> 32.4 mm, vias 2 -> 0
- net IO2: track 0.00 -> 17.6 mm, vias 0 -> 1
- net IO27: track 21.8 -> 4.92 mm
- net IO0: track 1.13 -> 15.6 mm, vias 0 -> 1
- net MOTOR: track 0.00 -> 12.8 mm, vias 0 -> 2
- net SCREEN_DC: track 21.2 -> 11.9 mm
- net N$10: track 0.00 -> 7.63 mm, vias 0 -> 1
- net SPI_CLK: track 19.8 -> 12.3 mm
- net N$3: track 0.00 -> 5.84 mm, vias 0 -> 1
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Other:
- outline, holes or cut-outs redrawn
- board text added: "trigotoram@gmail.com"
