File: PCB_Eagle/vA-ESP32.brd (EAGLE design)
At the start: 15 x 35 mm, 63 parts, among them Q2 IRLML0030, Q3 IRLML0030, U1 LTC4054, U2 MCP170x-3.3, U3 ESP32, U4 LIS3DH, U5 25Q32, X1 PCB, X2 I2C-SMD-SWATCH-I2C-5, X3 PCB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

Commit message: v
Parts:
- CP6, CP7: device !ht3_connectors:CP-1-C08MM -> !ht3_connectors:CP-1-C24MM
- moved LOGO1 14.7 mm to (9.40, 18.4)
- moved C14 5.32 mm to (1.80, 4.80)
- moved C23 3.14 mm to (5.70, 20.6), turned to 270 degrees
- moved C22 2.84 mm to (4.10, 23.0), turned to 180 degrees
- moved CP7 1.00 mm to (5.00, 1.50)
- moved C12 0.54 mm to (0.60, 6.20)
- moved CP6 0.40 mm to (10.6, 1.50)
- moved C18 0.40 mm to (12.4, 24.7)
- moved CP3 0.32 mm to (1.00, 12.6)
- moved C3 0.30 mm to (3.30, 3.30)
- moved CP8 0.28 mm to (5.30, 2.80)
- moved C8 0.20 mm to (3.30, 1.40)
- moved RA1 0.20 mm to (7.50, 1.40)
- moved U2 0.20 mm to (12.4, 27.3)
- moved CP9 0.14 mm to (9.10, 3.70)
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Connections:
- net IO0: no longer RA2.4
Routing:
- net IO0: track 28.9 -> 1.47 mm, vias 2 -> 0
- net GND: track 35.9 -> 43.2 mm, vias 37 -> 46
- net /IRQ: track 27.9 -> 31.3 mm
- net VDD: track 89.3 -> 86.2 mm
- net IO26: track 21.7 -> 23.5 mm
- net EN: track 11.3 -> 9.51 mm
- net SCREEN_CS: track 22.1 -> 21.1 mm
- net I39: track 3.55 -> 2.61 mm
- net I38: track 2.73 -> 3.43 mm
Other:
- board text added: "+"
- board text added: "-"
- board text added: "110"
