File: PCB_Eagle/vA-ESP32.sch (EAGLE design)
At the start: 68 parts, among them U1 25Q32, U14 ESP32, U18 M24SR04, U2 LTC4054, U8 LIS3DH, U9 MCP170x-3.0, X3 I2C-SMD-SWATCH-I2C-5, Y1 32.768, Y2 26MHz

Commit message: v
Parts:
- removed CP5, CP6: (no value), !ht3_connectors:CP
- removed D1: BAT54C-SOT323, !ht3_diode:BAT54C-SOT323
- removed D2: BAT54A-SOT323, !ht3_diode:BAT54A-SOT323
- removed LCD1: (no value), !ht3_modules:OLED_UG-2832HSWEG02
- removed R19: 10K, !ht3_passive:R-EU0603
- removed R20, R21: 4.7K, !ht3_passive:R-EU0603
- removed R5: 0, !ht3_passive:R-EU0402
- removed R6: 100, !ht3_passive:R-EU0402
- removed U18: M24SR04, !ht3_ic:M24SR04
- added C11, C5: 270pF, !ht3_passive:C-EU-C0603
- added C12: 100nF, !ht3_passive:C-EU-C0603
- added C16, C18: 270pF, !ht3_passive:C-EU-C0805
- added LOGO1: LOGO6, !ht3_misc:LOGO6
- added Q4: IRLML6401TR, !ht3_transistor:FET_P-SOT23
- added VD1: (no value), !ht3_diode:DIODESOD523
- C1: device !ht3_passive:C-EU-C0402 -> !ht3_passive:C-EU-C0603
- C40: value 10nF -> 100nF; device !ht3_passive:C-EU-C0603 -> !ht3_passive:C-EU-C0402
- D3: value 5.1V -> SS34; device !ht3_diode:ZENER-DIODESOD80C -> !ht3_diode:SCHOTTKY-DIODE-SOD123
- R4: value 0 -> 560K; device !ht3_passive:R-EU0402 -> !ht3_passive:R-EU0603
Connections:
- removed net IO26: U14.(DAC2/ADC2:9/RTC7)GPIO26
- removed net N$21: CP5.C1, D1.A1, D2.K2
- removed net N$24: CP6.C1, D1.A2, D2.K1
- removed net N$28: RA3.7, RA3.8
- removed net N$33: U18.RF-DIS
- removed net N$70: U18.AC1
- removed net N$71: U18.AC0
- removed net N$8: U18.GPO
- removed net SCREEN_LED: Q2.G, R21.2, RA3.3, U14.(ADC2:2/TOUCH2/RTC12/SPIWP)GPIO2
- new net IO2: Q2.G, RA3.3, U14.(ADC2:2/TOUCH2/RTC12/SPIWP)GPIO2
- new net N$10: C5.2, OLED1.C2P
- new net N$11: C12.1, C18.1, OLED1.VCC
- new net N$12: C16.1, OLED1.VCOMH
- new net N$14: OLED1.IREF, R4.2
- new net VBAT1: Q4.D
- net +5V: now also D3.A, Q4.G; no longer D3.C, R6.2
- net EN: now also RA3.1; no longer R19.2
- net GND: now also C12.2, C16.2, C18.2, OLED1.VSS, R4.1; no longer D2.AA, D3.A, R21.1, U18.VSS
- net I2C_SCL: now also OLED1.SCL; no longer U18.SCL
- net I2C_SDA: now also OLED1.SDA; no longer U18.SDA
- net IO0: now also RA4.4; no longer R20.1
- net MOTOR: now also U14.(DAC2/ADC2:9/RTC7)GPIO26
- net N$1: now also C11.2, OLED1.C1P; no longer R4.2, U14.32K_XP(GPIO32/ADC1:4/TOUCH9/RTC9)
- net N$22: now also VD1.A
- net N$23: now also VD1.C
- net N$3: now also C11.1, OLED1.C1N; no longer D1.CC, R6.1
- net N$5: now also C5.1, OLED1.C2N; no longer R5.2, U14.32K_XN(GPIO33/ADC1:5/TOUCH8/RTC8)
- net OSC32_I: now also U14.32K_XP(GPIO32/ADC1:4/TOUCH9/RTC9); no longer R4.1
- net OSC32_O: now also U14.32K_XN(GPIO33/ADC1:5/TOUCH8/RTC8); no longer R5.1
- net SCREEN_RES: now also OLED1.RES
- net VBAT: now also D3.C, Q4.S
- net VBAT_ADC: no longer U14.VDET_1(GPI34/ADC1:6)
- net VDD: now also OLED1.VBAT, OLED1.VDD, RA3.7, RA3.8, RA4.5; no longer R19.1, R20.2, U18.VCC
Other:
- moved on the sheet: C1, C10, C13, C14, C15, C17, C2, C25, C27, C3, C4, C40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

Commit message: v
Parts:
- removed C40, C51: 100nF, !ht3_passive:C-EU-C0402
- removed C42, C43: 270pF, !ht3_passive:C-EU-C0402
- removed C47: 3.9pF, !ht3_passive:C-EU-C0402
- removed C49: 2.4pF, !ht3_passive:C-EU-C0402
- removed CP10, CP11: (no value), !ht3_connectors:CP
- removed D3: SS34, !ht3_diode:SCHOTTKY-DIODE-SOD123
- removed Q4: IRLML6401TR, !ht3_transistor:FET_P-SOT23
- removed R10: 100, !ht3_passive:R-EU0603
- removed R11: 1M/10%, !ht3_passive:R-EU0402
- removed RA3, RA4: 10K, !ht3_passive:R-ARRAY-4X0402
- removed U9: MCP170x-3.0, !ht3_ic:MCP170XSOT23
- added C19: 2.2uFx16V, !ht3_passive:C-EU-C0805
- added C20, C21: 1uFx16V, !ht3_passive:C-EU-C0603
- added C22: 4.7uFx16V, !ht3_passive:C-EU-C0805
- added C23: 1uF, !ht3_passive:C-EU-C0402
- added C24: 100nF, !ht3_passive:C-EU-C0603
- added CP5, CP6: (no value), !ht3_connectors:CP
- added D1: SS34, !ht3_diode:SCHOTTKY-DIODE-SOD123
- added Q3: (no value), !ht3_transistor:FET_NSOT23
- added R7, R8: 100, !ht3_passive:R-EU0603
- added RA1, RA2: 10K, !ht3_passive:R-ARRAY-4X0402
- added U5: 25Q32, !ht3_ic:25CXX-USON8-2X3
- C1: value 100nF -> 10pF; device !ht3_passive:C-EU-C0603 -> !ht3_passive:C-EU-C0402
- C11: device !ht3_passive:C-EU-C0603 -> !ht3_passive:C-EU-C0402
- C12: value 100nF -> 270pF; device !ht3_passive:C-EU-C0603 -> !ht3_passive:C-EU-C0402
- C13: value 1uF -> 100nF; device !ht3_passive:C-EU-C0402 -> !ht3_passive:C-EU-C0603
- C14, C15: value 10pF -> 100nF
- C16: value 270pF -> 10nF; device !ht3_passive:C-EU-C0805 -> !ht3_passive:C-EU-C0402
- C17: value 100nF -> 3nF
- C18: value 270pF -> 4.7uF; device !ht3_passive:C-EU-C0805 -> !ht3_passive:C-EU-C0603
- C2, C4: value 4.7uF -> 10pF; device !ht3_passive:C-EU-C0603 -> !ht3_passive:C-EU-C0402
- C25: value 10nF -> 100nF
- C3: value 3nF -> 4.7uF; device !ht3_passive:C-EU-C0402 -> !ht3_passive:C-EU-C0603
- C5: value 270pF -> 100nF; device !ht3_passive:C-EU-C0603 -> !ht3_passive:C-EU-C0402
- C7: value 4.7uF -> 2.4pF; device !ht3_passive:C-EU-C0603 -> !ht3_passive:C-EU-C0402
- C8: value 10pF -> 3.9pF
- C9: value 100nF -> 4.7uF; device !ht3_passive:C-EU-C0402 -> !ht3_passive:C-EU-C0603
- CP1: device !ht3_connectors:CP -> !ht3_connectors:CP-1
- CP3: device !ht3_connectors:CP-1 -> !ht3_connectors:CP
- Q1: value (none) -> IRLML6401TR; device !ht3_transistor:FET_NSOT23 -> !ht3_transistor:FET_P-SOT23
- R1: value 10K -> 1M/10%
- R2: value 100 -> 10K; device !ht3_passive:R-EU0603 -> !ht3_passive:R-EU0402
- R4: value 560K -> 390-560K
- R6: value 100K -> 1M
- U1: value 25Q32 -> LTC4054; device !ht3_ic:25CXX-USON8-2X3 -> !ht3_ic:LTC4054
- U2: value LTC4054 -> MCP170x-3.0; device !ht3_ic:LTC4054 -> !ht3_ic:MCP170XSOT23
- X2: value (none) -> I2C-SMD-SWATCH-I2C-5; device !ht3_connectors:CON-2PSMD-2 -> !ht3_connectors:I2C-SMD-SWATCH-I2C-5
- X3: value I2C-SMD-SWATCH-I2C-5 -> (none); device !ht3_connectors:I2C-SMD-SWATCH-I2C-5 -> !ht3_connectors:CON-2PSMD-2
- renumbered C27 to C26, L7 to L1, R12 to R5, R13 to R6, U14 to U3, U8 to U4
Connections:
- removed net VBAT1: Q4.D
- new net N$13: D1.C, Q1.S, U2.VIN
- net +5V: now also C3.1, CP2.C1, D1.A, Q1.G, U1.VCC; no longer C2.1, CP3.C1, D3.A, Q4.G, U2.VCC
- net /INT: now also RA1.3; no longer RA4.3
- net ANT: now also C7.1, C8.1, CP3.C1; no longer C47.1, C49.1, CP4.C1
- net EN: now also C5.1, CP8.C1, RA2.1; no longer C40.1, CP10.C1, RA3.1
- net GND: now also C19.2, C22.2, C23.2, C24.2, C3.2, C5.2, CP1.C1, Q3.S, R2.2, RA2.6, U1.GND, U5.VSS, X2.GND; no longer C12.2, C17.2, C40.2, C49.2, C51.2, C8.2, CP2.C1, Q1.S, R1.2, RA3.6, U1.VSS, U9.GND, X3.GND
- net I2C_SCL: now also RA1.1, X2.SCL; no longer RA4.1, X3.SCL
- net I2C_SDA: now also RA1.2, X2.SDA; no longer RA4.2, X3.SDA
- net I36: now also C11.1; no longer C43.1
- net I37: now also C11.2; no longer C43.2
- net I38: now also C12.1; no longer C42.1
- net I39: now also C12.2; no longer C42.2
- net IO0: now also CP9.C1, RA1.4; no longer CP11.C1, RA4.4
- net IO1: now also CP4.C1; no longer CP7.C1
- net IO10: now also U5./WP/IO2; no longer U1./WP/IO2
- net IO11: now also U5./CS; no longer U1./CS
- net IO2: now also RA2.3; no longer RA3.3
- net IO27: now also CP7.C1; no longer CP1.C1
- net IO3: now also CP5.C1; no longer CP8.C1
- net IO4: now also CP6.C1; no longer CP9.C1
- net IO6: now also U5.SCK; no longer U1.SCK
- net IO7: now also U5.SO/IO1; no longer U1.SO/IO1
- net IO8: now also U5.SI/IO0; no longer U1.SI/IO0
- net IO9: now also U5./HOLD/IO3; no longer U1./HOLD/IO3
- net MOTOR: now also Q3.G; no longer Q1.G
- net N$1: now also C21.2; no longer C11.2
- net N$10: now also C20.2; no longer C5.2
- net N$11: now also C22.1, C24.1; no longer C12.1, C18.1
- net N$12: now also C19.1; no longer C16.1
- net N$17: now also R7.2; no longer R10.2
- net N$2: now also C17.1; no longer C3.1
- net N$22: now also Q3.D, X3.2; no longer Q1.D, X2.2
- net N$23: now also R8.2, X3.1; no longer R2.2, X2.1
- net N$3: now also C21.1; no longer C11.1
- net N$4: now also C16.1, C17.2; no longer C25.1, C3.2
- net N$5: now also C20.1; no longer C5.1
- net N$6: now also R2.1, U1.PROG; no longer R1.1, U2.PROG
- net N$7: now also C8.2; no longer C47.2
- net N$9: now also R7.1; no longer R10.1
- net OSC26_I: now also C1.1, R1.1; no longer C14.1, R11.1
- net OSC26_O: now also C6.1, R1.2; no longer C15.1, R11.2
- net OSC32_I: now also C2.1; no longer C8.1
- net OSC32_O: now also C4.1; no longer C6.1
- net VBAT: now also C9.1, Q1.D, R8.1, U1.BAT; no longer C4.1, D3.C, Q4.S, R2.1, U2.BAT, U9.VIN
- net VBAT_ADC: now also C25.1; no longer C17.1
- net VDD: now also C14.1, C15.1, C18.1, C23.1, RA1.5, RA1.6, RA1.7, RA1.8, RA2.7, RA2.8, U2.VOUT\, X2.VCC; no longer C1.1, C51.1, C7.1, C9.1, RA3.7, RA3.8, RA4.5, RA4.6, RA4.7, RA4.8, U9.VOUT\, X3.VCC
- net VDD_SDIO: now also U5.VCC; no longer U1.VCC
Other:
- note removed: ""BOOT""
- note removed: "I2C memory in SOT-6 !!!"
- note removed: "MAX9814"
- note removed: "http://doc.satoshilabs.com/trezor-tech/api.html"
- note removed: "http://elm-chan.org/works/sd8p/report.html"
- note removed: "http://vrtp.ru/index.php?act=categories&CODE=article&article=3437"
- note removed: "http://vrtp.ru/screenshots/3410_schema.pdf"
- note removed: "http://www.atmel.com/images/doc32110.pdf"
- note removed: "https://bitcointalk.org/index.php?topic=78614.0"
- note removed: "https://esp8266.ru/forum/threads/wiieva-esp8266-stm32-v-formfaktore-arduino.1511/"
- note removed: "https://geektimes.ru/post/285016/"
- note removed: "https://geektimes.ru/post/286650/"
- note removed: "https://github.com/digitalbitbox/mcu/tree/master/src"
- note removed: "https://github.com/satoshilabs/docs"
- note removed: "https://github.com/trezor/"
- note removed: "https://habrahabr.ru/post/323598/"
- note removed: "https://hackaday.io/project/18014-5-alphabets-charlieplexed-matrix-display-22x5"
- note removed: "https://hackaday.io/project/5511-scrolled-watch"
- note removed: "https://perso.aquilenet.fr/~sven337/english/2016/07/14/DIY-wifi-baby-monitor.html"
- note removed: "nfc"
- note removed: "Выяснить сколько тока потребляет ЛДО + часы 2. Выяснить с подключением сз2012"
- moved on the sheet: C1, C10, C11, C12, C13, C14, C15, C16, C17, C18, C2, C25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

Commit message: v
Parts:
- C19: value 2.2uFx16V -> 1uFx16V; device !ht3_passive:C-EU-C0805 -> !ht3_passive:C-EU-C0603
- C2, C4: value 10pF -> 12pF
- C21: value 1uFx16V -> 2.2uFx16V; device !ht3_passive:C-EU-C0603 -> !ht3_passive:C-EU-C0805
- C23: value 1uF -> 100nF; device !ht3_passive:C-EU-C0402 -> !ht3_passive:C-EU-C0603
- C24: value 100nF -> 1uF; device !ht3_passive:C-EU-C0603 -> !ht3_passive:C-EU-C0402
- C5: value 100nF -> 10pF
- C6: value 10pF -> 100nF
- CP1: value (none) -> GND
- CP2: value (none) -> +5V
- CP3: value (none) -> ANT
- CP4: value (none) -> TX
- CP5: value (none) -> RX
- CP6: value (none) -> TL
- CP7: value (none) -> TR
- CP8: value (none) -> RESET
- CP9: value (none) -> BOOT
- D1: value SS34 -> NF
- Q2, Q3: value (none) -> IRLML0030
- R7, R8: value 100 -> 10
- U2: value MCP170x-3.0 -> MCP170x-3.3
- VD1: value (none) -> 4148
- X1, X3: value (none) -> PCB
Connections:
- removed net /INT: RA1.3
- removed net IO17: U3.(HS1_DATA5)GPIO17
- removed net IO25: U3.(DAC1/ADC2:8/RTC6)GPIO25
- removed net JTAG_TCK: U3.(GPIO13/ADC2:4/TOUCH4/RTC14/SPID/U0CTS)MTCK
- removed net JTAG_TDI: U3.(GPIO12/ADC2:5/TOUCH5/RTC15/SPIQ)MTDI
- removed net JTAG_TDO: U3.(GPIO15/ADC2:3/TOUCH3/RTC13/SPICSO/U0RTS)MTDO
- removed net JTAG_TMS: U3.(GPIO14/ADC2:6/TOUCH6/RTC16/SPICLK)MTMS
- removed net MOTOR: Q3.G, U3.(DAC2/ADC2:9/RTC7)GPIO26
- new net IO26: Q2.G, RA2.3, U3.(DAC2/ADC2:9/RTC7)GPIO26
- net /IRQ: now also RA1.3
- net EN: now also C6.1, RA2.4; no longer C5.1, RA2.1
- net GND: now also C21.2, RA2.8; no longer C19.2
- net IO2: now also Q3.G, RA2.1; no longer Q2.G, RA2.3
- net N$1: now also C20.2; no longer C21.2
- net N$10: now also C19.2; no longer C20.2
- net N$11: now also C23.1; no longer C24.1
- net N$12: now also C21.1; no longer C19.1
- net N$13: now also C9.1
- net N$3: now also C20.1; no longer C21.1
- net N$5: now also C19.1; no longer C20.1
- net OSC26_O: now also C5.1; no longer C6.1
- net VBAT: no longer C9.1
- net VDD: now also C24.1, RA2.5; no longer C23.1, RA2.7, RA2.8
Other:
- note added: "BATT"
- note added: "MOTOR"
- note added: "Touch Left button"
- note added: "Touch Right button"
- note added: "WIFI/BLE"
- note added: "to external Pulse/Oximeter"
- note removed: "WIFI"
- moved on the sheet: C1, C10, C11, C12, C13, C14, C15, C16, C17, C18, C19, C2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

Commit message: v
Parts:
- removed D1: NF, !ht3_diode:SCHOTTKY-DIODE-SOD123
- removed Q1: IRLML6401TR, !ht3_transistor:FET_P-SOT23
- C10: value 100nF -> 2.4pF
- C11: value 270pF -> 3.9pF
- C13: value 100nF -> 270pF; device !ht3_passive:C-EU-C0603 -> !ht3_passive:C-EU-C0402
- C15: value 100nF -> 10nF
- C16: value 10nF -> 4.7uF; device !ht3_passive:C-EU-C0402 -> !ht3_passive:C-EU-C0603
- C2: value 12pF -> 100nF
- C3: value 4.7uF -> 12pF; device !ht3_passive:C-EU-C0603 -> !ht3_passive:C-EU-C0402
- C4: value 12pF -> 4.7uF; device !ht3_passive:C-EU-C0402 -> !ht3_passive:C-EU-C0603
- C5: value 10pF -> 100nF; device !ht3_passive:C-EU-C0402 -> !ht3_passive:C-EU-C0603
- C7: value 2.4pF -> 100nF
- C8: value 3.9pF -> 12pF
- C9: value 4.7uF -> 10pF; device !ht3_passive:C-EU-C0603 -> !ht3_passive:C-EU-C0402
Connections:
- removed net N$13: C9.1, D1.C, Q1.S, U2.VIN
- net +5V: now also C4.1; no longer C3.1, D1.A, Q1.G
- net /IRQ: no longer RA1.3
- net ANT: now also C10.1, C11.1; no longer C7.1, C8.1
- net EN: now also C14.1, RA1.5; no longer C6.1, RA2.4
- net GND: now also C8.2, RA1.2, RA1.6, RA1.7, RA1.8; no longer C13.2, RA2.6, RA2.8
- net I2C_SCL: now also RA2.1; no longer RA1.1
- net I2C_SDA: now also RA2.2; no longer RA1.2
- net I36: now also C12.1; no longer C11.1
- net I37: now also C12.2; no longer C11.2
- net I38: now also C13.1; no longer C12.1
- net I39: now also C13.2; no longer C12.2
- net IO0: now also RA2.4; no longer RA1.4
- net IO2: now also RA1.1; no longer RA2.1
- net IO26: now also RA1.3; no longer RA2.3
- net N$4: now also C15.1; no longer C16.1
- net N$7: now also C11.2; no longer C8.2
- net OSC26_O: now also C9.1; no longer C5.1
- net OSC32_I: now also C3.1; no longer C2.1
- net OSC32_O: now also C8.1; no longer C4.1
- net VBAT: now also C16.1, U2.VIN; no longer Q1.D
- net VDD: now also C2.1, C5.1, C6.1, C7.1, RA1.4, RA2.6, RA2.7, RA2.8; no longer C10.1, C13.1, C14.1, C15.1, RA1.5, RA1.6, RA1.7, RA1.8
Other:
- note added: "??"
- moved on the sheet: C10, C11, C12, C13, C14, C15, C16, C2, C3, C4, C5, C6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

Commit message: v
Parts:
- CP6, CP7: device !ht3_connectors:CP -> !ht3_connectors:CP-CP-1-C25
Connections:
- net IO0: no longer RA2.4
Changed lines of the file:
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@@
 <grid distance="0.1" unitdist="inch" unit="inch" style="lines" multiple="1" display="no" altdistance="0.01" altunitdist="inch" altunit="inch"/>
 <layers>
-<layer number="1" name="Top" color="12" fill="1" visible="no" active="no"/>
-<layer number="2" name="Route2" color="1" fill="3" visible="no" active="no"/>
-<layer number="3" name="Route3" color="4" fill="3" visible="no" active="no"/>
-<layer number="4" name="Route4" color="1" fill="4" visible="no" active="no"/>
-<layer number="5" name="Route5" color="4" fill="4" visible="no" active="no"/>
-<layer number="6" name="Route6" color="1" fill="8" visible="no" active="no"/>
-<layer number="7" name="Route7" color="4" fill="8" visible="no" active="no"/>
-<layer number="8" name="Route8" color="1" fill="2" visible="no" active="no"/>
-<layer number="9" name="Route9" color="4" fill="2" visible="no" active="no"/>
-<layer number="10" name="Route10" color="1" fill="7" visible="no" active="no"/>
-<layer number="11" name="Route11" color="4" fill="7" visible="no" active="no"/>
-<layer number="12" name="Route12" color="1" fill="5" visible="no" active="no"/>
-<layer number="13" name="Route13" color="4" fill="5" visible="no" active="no"/>
-<layer number="14" name="Route14" color="1" fill="6" visible="no" active="no"/>
-<layer number="15" name="Route15" color="4" fill="6" visible="no" active="no"/>
-<layer number="16" name="Bottom" color="1" fill="1" visible="no" active="no"/>
-<layer number="17" name="Pads" color="2" fill="1" visible="no" active="no"/>
-<layer number="18" name="Vias" color="2" fill="1" visible="no" active="no"/>
-<layer number="19" name="Unrouted" color="6" fill="1" visible="no" active="no"/>
-<layer number="20" name="Dimension" color="15" fill="1" visible="no" active="no"/>
-<layer number="21" name="tPlace" color="7" fill="1" visible="no" active="no"/>
-<layer number="22" name="bPlace" color="7" fill="1" visible="no" active="no"/>
-<layer number="23" name="tOrigins" color="15" fill="1" visible="no" active="no"/>
-<layer number="24" name="bOrigins" color="15" fill="1" visible="no" active="no"/>
-<layer number="25" name="tNames" color="24" fill="1" visible="no" active="no"/>
-<layer number="26" name="bNames" color="24" fill="1" visible="no" active="no"/>
-<layer number="27" name="tValues" color="7" fill="1" visible="no" active="no"/>
-<layer number="28" name="bValues" color="7" fill="1" visible="no" active="no"/>
+<layer number="1" name="Top" color="12" fill="1" visible="yes" active="no"/>
+<layer number="2" name="Route2" color="1" fill="3" visible="yes" active="no"/>
+<layer number="3" name="Route3" color="4" fill="3" visible="yes" active="no"/>
+<layer number="4" name="Route4" color="1" fill="4" visible="yes" active="no"/>
+<layer number="5" name="Route5" color="4" fill="4" visible="yes" active="no"/>
+<layer number="6" name="Route6" color="1" fill="8" visible="yes" active="no"/>
+<layer number="7" name="Route7" color="4" fill="8" visible="yes" active="no"/>
+<layer number="8" name="Route8" color="1" fill="2" visible="yes" active="no"/>
+<layer number="9" name="Route9" color="4" fill="2" visible="yes" active="no"/>
+<layer number="10" name="Route10" color="1" fill="7" visible="yes" active="no"/>
+<layer number="11" name="Route11" color="4" fill="7" visible="yes" active="no"/>
+<layer number="12" name="Route12" color="1" fill="5" visible="yes" active="no"/>
+<layer number="13" name="Route13" color="4" fill="5" visible="yes" active="no"/>
+<layer number="14" name="Route14" color="1" fill="6" visible="yes" active="no"/>
+<layer number="15" name="Route15" color="4" fill="6" visible="yes" active="no"/>
+<layer number="16" name="Bottom" color="1" fill="1" visible="yes" active="no"/>
+<layer number="17" name="Pads" color="2" fill="1" visible="yes" active="no"/>
+<layer number="18" name="Vias" color="2" fill="1" visible="yes" active="no"/>
+<layer number="19" name="Unrouted" color="6" fill="1" visible="yes" active="no"/>
+<layer number="20" name="Dimension" color="15" fill="1" visible="yes" active="no"/>
+<layer number="21" name="tPlace" color="7" fill="1" visible="yes" active="no"/>
+<layer number="22" name="bPlace" color="7" fill="1" visible="yes" active="no"/>
+<layer number="23" name="tOrigins" color="15" fill="1" visible="yes" active="no"/>
+<layer number="24" name="bOrigins" color="15" fill="1" visible="yes" active="no"/>
+<layer number="25" name="tNames" color="24" fill="1" visible="yes" active="no"/>
+<layer number="26" name="bNames" color="24" fill="1" visible="yes" active="no"/>
+<layer number="27" name="tValues" color="7" fill="1" visible="yes" active="no"/>
+<layer number="28" name="bValues" color="7" fill="1" visible="yes" active="no"/>
 <layer number="29" name="tStop" color="7" fill="3" visible="no" active="no"/>
 <layer number="30" name="bStop" color="7" fill="6" visible="no" active="no"/>
@@
 <layer number="35" name="tGlue" color="7" fill="4" visible="no" active="no"/>
 <layer number="36" name="bGlue" color="7" fill="5" visible="no" active="no"/>
-<layer number="37" name="tTest" color="7" fill="1" visible="no" active="no"/>
-<layer number="38" name="bTest" color="7" fill="1" visible="no" active="no"/>
+<layer number="37" name="tTest" color="7" fill="1" visible="yes" active="no"/>
+<layer number="38" name="bTest" color="7" fill="1" visible="yes" active="no"/>
 <layer number="39" name="tKeepout" color="4" fill="11" visible="no" active="no"/>
 <layer number="40" name="bKeepout" color="1" fill="11" visible="no" active="no"/>
@@
 <layer number="44" name="Drills" color="7" fill="1" visible="no" active="no"/>
 <layer number="45" name="Holes" color="7" fill="1" visible="no" active="no"/>
-<layer number="46" name="Milling" color="3" fill="1" visible="no" active="no"/>
-<layer number="47" name="Measures" color="13" fill="1" visible="no" active="no"/>
-<layer number="48" name="Document" color="7" fill="1" visible="no" active="no"/>
-<layer number="49" name="Reference" color="7" fill="1" visible="no" active="no"/>
-<layer number="50" name="dxf" color="7" fill="1" visible="no" active="no"/>
-<layer number="51" name="tDocu" color="9" fill="1" visible="no" active="no"/>
-<layer number="52" name="bDocu" color="14" fill="1" visible="no" active="no"/>
-<layer number="53" name="tGND_GNDA" color="7" fill="9" visible="no" active="no"/>
-<layer number="54" name="bGND_GNDA" color="1" fill="9" visible="no" active="no"/>
-<layer number="56" name="wert" color="7" fill="1" visible="no" active="no"/>
-<layer number="57" name="tCAD" color="7" fill="1" visible="no" active="no"/>
-<layer number="59" name="tCarbon" color="7" fill="1" visible="no" active="no"/>
-<layer number="60" name="bCarbon" color="7" fill="1" visible="no" active="no"/>
+<layer number="46" name="Milling" color="3" fill="1" visible="yes" active="no"/>
+<layer number="47" name="Measures" color="13" fill="1" visible="yes" active="no"/>
+<layer number="48" name="Document" color="7" fill="1" visible="yes" active="no"/>
+<layer number="49" name="Reference" color="7" fill="1" visible="yes" active="no"/>
+<layer number="50" name="dxf" color="7" fill="1" visible="yes" active="no"/>
+<layer number="51" name="tDocu" color="9" fill="1" visible="yes" active="no"/>
+<layer number="52" name="bDocu" color="14" fill="1" visible="yes" active="no"/>
+<layer number="53" name="tGND_GNDA" color="7" fill="9" visible="yes" active="no"/>
+<layer number="54" name="bGND_GNDA" color="1" fill="9" visible="yes" active="no"/>
+<layer number="56" name="wert" color="7" fill="1" visible="yes" active="no"/>
+<layer number="57" name="tCAD" color="7" fill="1" visible="yes" active="no"/>
+<layer number="59" name="tCarbon" color="7" fill="1" visible="yes" active="no"/>
+<layer number="60" name="bCarbon" color="7" fill="1" visible="yes" active="no"/>
 <layer number="88" name="SimResults" color="9" fill="1" visible="no" active="yes"/>
 <layer number="89" name="SimProbes" color="9" fill="1" visible="no" active="yes"/>
@@
 <part name="CP8" library="!ht3_connectors" deviceset="CP" device="" value="RESET"/>
 <part name="CP9" library="!ht3_connectors" deviceset="CP" device="" value="BOOT"/>
-<part name="CP7" library="!ht3_connectors" deviceset="CP" device="" value="TR"/>
-<part name="CP6" library="!ht3_connectors" deviceset="CP" device="" value="TL"/>
+<part name="CP7" library="!ht3_connectors" deviceset="CP" device="-CP-1-C25" value="TR"/>
+<part name="CP6" library="!ht3_connectors" deviceset="CP" device="-CP-1-C25" value="TL"/>
 <part name="C5" library="!ht3_passive" deviceset="C-EU" device="-C0603" value="100nF"/>
 <part name="GND6" library="!ht3_misc" deviceset="GND" device=""/>
@@
 <pinref part="RA2" gate="G$1" pin="5"/>
 <wire x1="-33.02" y1="45.72" x2="-35.56" y2="45.72" width="0.1524" layer="91"/>
+<wire x1="-35.56" y1="38.1" x2="-33.02" y2="38.1" width="0.1524" layer="91"/>
+<wire x1="-33.02" y1="38.1" x2="-33.02" y2="45.72" width="0.1524" layer="91"/>
+<junction x="-33.02" y="45.72"/>
 </segment>
 <segment>
@@
 </segment>
 <segment>
-<pinref part="RA2" gate="G$1" pin="4"/>
-<wire x1="-48.26" y1="45.72" x2="-50.8" y2="45.72" width="0.1524" layer="91"/>
-<label x="-50.8" y="45.72" size="1.27" layer="95" font="vector" rot="R180" xref="yes"/>
-</segment>
-</net>
+<label x="-48.26" y="38.1" size="1.27" layer="95" font="vector" rot="R180" xref="yes"/>
+<wire x1="-45.72" y1="38.1" x2="-48.26" y2="38.1" width="0.1524" layer="91"/>
+</segment>
+</net>
